File: anlg1v/anlg1v.kicad_pcb (KiCad board)
At the start: 2 copper layers, 188 x 93.5 mm, 118 parts, among them J1 PJ-007, J2 AudioJack3, J3 AudioJack3, J4 USB_B, SW1 Disp_back, SW10 Disp_Scroll/Sel, SW4 Env_Sel, SW5 VCO_On/Off, SW6 Digiosc_On/Off, SW9 LFO_Freq/Sel, U1 SSI2131, U10 MCP6004, U11 SSI2164, U12 6N138, U13 MCP2221AxSL, U14 CD4051B, U15 CD4051B, U16 CD4051B, U17 CD4052B, U2 Teensy4.0, U3 MCP4922, U4 LT1962-2.5, U5 MCP6004, U6 CD4052B, U7 SSI2144, U8 MCP4922, U9 CD4051B

Commit message: Add files via upload
Parts:
- added R30: 22k, Resistor_SMD:R_0603_1608Metric, F.Cu at (0.00, 0.00)
- added R31: 100k, Resistor_SMD:R_0603_1608Metric, B.Cu at (0.00, 0.00)
- R25: value 1k -> 20k
- moved C4 288.5 mm to (0.00, 0.00)
- moved REF** 288.1 mm to (0.00, 0.00)
- moved U4 286.5 mm to (0.00, 0.00)
- moved PS1 282.8 mm to (0.00, 0.00), turned to 0 degrees
- moved C1 279.9 mm to (0.00, 0.00), turned to 0 degrees
- moved J1 279.7 mm to (0.00, 0.00), turned to 0 degrees
- moved C7 278.2 mm to (0.00, 0.00), turned to 0 degrees
- moved C6 277.3 mm to (0.00, 0.00), turned to 0 degrees
- moved R2 276.4 mm to (0.00, 0.00), turned to 0 degrees
- moved R3 275.7 mm to (0.00, 0.00), turned to 0 degrees
- moved Env1_Dest1 274.5 mm to (0.00, 0.00), turned to 0 degrees
- moved REF** 273.5 mm to (0.00, 0.00)
- moved C5 270.4 mm to (0.00, 0.00)
- moved C3 269.7 mm to (0.00, 0.00), turned to 0 degrees
- moved C2 266.6 mm to (0.00, 0.00), turned to 0 degrees
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Connections:
- C21 pad 1: Net-(U5C-+) -> Net-(U5C--)
- C4 pad 2: GND -> Net-(U4-BYP)
- J4 pad 5: GND -> (no net)
- R25 pad 2: Net-(U5C-+) -> Net-(U5C--)
- U11 pad 4: Net-(U5C-+) -> Net-(U5C--)
- U14 pad 3: unconnected-(U14-X-Pad3) -> MUX1
- U15 pad 3: unconnected-(U15-X-Pad3) -> MUX2
- U16 pad 3: unconnected-(U16-X-Pad3) -> MUX3
- U2 pad 11: unconnected-(U2-9_OUT1C-Pad11) -> RotarySelA
- U2 pad 12: unconnected-(U2-10_CS_MQSR-Pad12) -> RotarySelB
- U2 pad 24: unconnected-(U2-17_A3_TX4_SDA1-Pad24) -> MUX1
- U2 pad 27: unconnected-(U2-20_A6_TX5_LRCLK1-Pad27) -> MUX2
- U2 pad 28: unconnected-(U2-21_A7_RX5_BCLK1-Pad28) -> MUX3
- U2 pad 29: unconnected-(U2-22_A8_CTX1-Pad29) -> RotaryOut2
- U2 pad 30: unconnected-(U2-23_A9_CRX1_MCLK1-Pad30) -> RotaryOut1
- U4 pad 3: GND -> Net-(U4-BYP)
- U5 pad 10: Net-(U5C-+) -> GND
- U5 pad 9: GND -> Net-(U5C--)
Routing:
- net RotaryOut2: track 0.00 -> 83.9 mm, vias 0 -> 8
- net RotaryOut1: track 0.00 -> 81.2 mm, vias 0 -> 4
- net RotarySelB: track 0.00 -> 59.2 mm, vias 0 -> 5
- net RotarySelA: track 0.00 -> 56.9 mm, vias 0 -> 3
- net Net-(U5C-+): track 42.8 -> 0.00 mm
- net Net-(U5C--): track 0.00 -> 38.4 mm, vias 0 -> 4
- net MUX3: track 0.00 -> 34.4 mm, vias 0 -> 2
- net MUX2: track 0.00 -> 27.2 mm, vias 0 -> 6
- net VCF_CV: track 1.27 -> 26.1 mm, vias 0 -> 3
- net GND: track 202.9 -> 227.1 mm, vias 65 -> 66
- net MUX1: track 0.00 -> 13.4 mm, vias 0 -> 1
- net RES_CV: track 1.27 -> 13.6 mm, vias 0 -> 2
- net Net-(U4-BYP): track 0.00 -> 6.99 mm, vias 0 -> 2
- net Net-(U7-Q_CTRL): track 20.1 -> 25.1 mm
- net Net-(U5B--): track 17.9 -> 21.6 mm, vias 0 -> 1
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